File: schematics/LucyLowLevelController.kicad_pcb (KiCad board)
At the start: 2 copper layers, 38 parts, among them IC1 ATMEGA328P-P, K1 Serial Interface Connector, K3 Power IN, P1 Servo PWM, P10 CONN_4X2, P2 Power Out ODROID, P3 CONN_1, P4 Servo Block, P5 CONN_1, P6 LED_CONN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

Commit message: .
Connections:
- D1 pad 2: N-0000032 -> Net-(D1-Pad2)
- IC1 pad 10: (no net) -> Net-(IC1-Pad10)
- IC1 pad 11: (no net) -> Net-(IC1-Pad11)
- IC1 pad 14: (no net) -> Net-(IC1-Pad14)
- IC1 pad 15: (no net) -> Net-(IC1-Pad15)
- IC1 pad 4: (no net) -> Net-(IC1-Pad4)
- P10 pad 4: (no net) -> /O-RXD
- P10 pad 5: (no net) -> /#204
- P10 pad 6: (no net) -> /O-TXD
- P10 pad 8: (no net) -> Net-(P10-Pad8)
- U1 pad 3: N-0000032 -> Net-(D1-Pad2)
Routing:
- net Net-(D1-Pad2): track 0.00 -> 17.8 mm, vias 0 -> 1
- net N-0000032: track 33.0 -> 15.2 mm, vias 2 -> 1
